File: Electronic/PCBWallet/PCBWallet.kicad_pcb (KiCad board)
At the start: 2 copper layers, 122.7 x 142 mm, 8 parts, among them U1 NFCTag_ST25DV

Commit message: finishing first version of PCBWallet
Parts:
- added G***: LOGO, Libary:lockcard_logo, F.Cu at (117.3, 135.0)
- added mouse-bite-2mm-slot: VAL**, Libary:mouse-bite-2mm-slot, F.Cu at (36.8, 60.0)
- added mouse-bite-2mm-slot: VAL**, Libary:mouse-bite-2mm-slot, F.Cu at (87.8, 51.5)
- added mouse-bite-2mm-slot: VAL**, Libary:mouse-bite-2mm-slot, F.Cu at (95.8, 146.0)
- added mouse-bite-2mm-slot: VAL**, Libary:mouse-bite-2mm-slot, F.Cu at (78.2, 146.0)
- added mouse-bite-2mm-slot: VAL**, Libary:mouse-bite-2mm-slot, F.Cu at (137.2, 146.0)
- added mouse-bite-2mm-slot: VAL**, Libary:mouse-bite-2mm-slot, F.Cu at (87.8, 154.4)
- added mouse-bite-2mm-slot: VAL**, Libary:mouse-bite-2mm-slot, F.Cu at (95.8, 60.0)
- added mouse-bite-2mm-slot: VAL**, Libary:mouse-bite-2mm-slot, F.Cu at (87.8, 127.5)
- added mouse-bite-2mm-slot: VAL**, Libary:mouse-bite-2mm-slot, F.Cu at (36.8, 146.0)
- added mouse-bite-2mm-slot: VAL**, Libary:mouse-bite-2mm-slot, F.Cu at (78.2, 60.0)
- added mouse-bite-2mm-slot: VAL**, Libary:mouse-bite-2mm-slot, F.Cu at (137.2, 60.0)
- added mouse-bite-2mm-slot: VAL**, Libary:mouse-bite-2mm-slot, F.Cu at (87.8, 78.4)
Other:
- board size 122.7 x 142 mm -> 116 x 142 mm

Commit message: start rev 2.0
Other:
- board size 116 x 142 mm -> 203.9 x 142 mm
